File: Ultra96-IO-Mezzanine.kicad_pcb (KiCad board)
At the start: 2 copper layers, 85 x 54 mm, 6 parts, among them P1 CONN_02X20, P2 CONN_02X20

Commit message: Initial commit
Parts:
- P2: footprint 96boards:Socket_Strip_SMD_2x20_Pitch2mm -> 96boards:Socket_Strip_Straight_2x20_Pitch2mm
