File: Ultra96-IO-Mezzanine.sch (KiCad schematic (older format))
At the start: 22 parts, among them J1 Conn_02x20_Odd_Even, J2 USB_C_Receptacle_USB2.0, P2 CONN_02X20, Q1 STL6P3LLH6, SW1 SW_Push, SW2 SW_Push, SW3 SW_SP3T, U1 TXS0108EPW, U2 TXS0108EPW, U3 AMS1117-3.3, U4 STUSB4500QTR

Commit message: Updated
Parts:
- added R5: 100K, symbol Ultra96-IO-Mezzanine-rescue:R-Device
- C1, C2, C3, C4: symbol Device:C -> Ultra96-IO-Mezzanine-rescue:C-Device
- D1, D2, D3: symbol Device:D_Schottky -> Ultra96-IO-Mezzanine-rescue:D_Schottky-Device
- J1: symbol Connector_Generic:Conn_02x20_Odd_Even -> Ultra96-IO-Mezzanine-rescue:Conn_02x20_Odd_Even-Connector_Generic
- J2: symbol Connector:USB_C_Receptacle_USB2.0 -> Ultra96-IO-Mezzanine-rescue:USB_C_Receptacle_USB2.0-Connector
- Q1: symbol STL6P3LLH6:STL6P3LLH6 -> Ultra96-IO-Mezzanine-rescue:STL6P3LLH6-STL6P3LLH6
- R1, R2, R3, R4: symbol Device:R -> Ultra96-IO-Mezzanine-rescue:R-Device
- SW1, SW2: symbol Switch:SW_Push -> Ultra96-IO-Mezzanine-rescue:SW_Push-Switch
- SW3: symbol Switch:SW_SP3T -> Ultra96-IO-Mezzanine-rescue:SW_SP3T-Switch
- U1, U2: symbol Logic_LevelTranslator:TXS0108EPW -> Ultra96-IO-Mezzanine-rescue:TXS0108EPW-Logic_LevelTranslator
- U3: symbol Regulator_Linear:AMS1117-3.3 -> Ultra96-IO-Mezzanine-rescue:AMS1117-3.3-Regulator_Linear
- U4: symbol Interface_USB:STUSB4500QTR -> Ultra96-IO-Mezzanine-rescue:STUSB4500QTR-Interface_USB
Connections:
- net GND: now also R5.2
- net GPIO_A: no longer J1.13 (Pin_13)
- net GPIO_B: no longer J1.15 (Pin_15)
- net GPIO_C: no longer J1.16 (Pin_16)
- net GPIO_D: no longer J1.18 (Pin_18)
- net GPIO_E: no longer J1.22 (Pin_22)
- net GPIO_F: no longer J1.37 (Pin_37)
- net GPIO_G: no longer J1.29 (Pin_29)
- net GPIO_H: no longer J1.31 (Pin_31)
- net GPIO_I: no longer J1.33 (Pin_33)
- net GPIO_J: no longer J1.35 (Pin_35)
- net GPIO_K: no longer J1.38 (Pin_38)
- net GPIO_L: no longer J1.40 (Pin_40)
- net I2C0_SCL: no longer J1.28 (Pin_28)
- net I2C0_SDA: no longer J1.27 (Pin_27)
- net I2C1_SCL: no longer J1.5 (Pin_5)
- net I2C1_SDA: no longer J1.3 (Pin_3)
- net SPIO_CS: no longer J1.24 (Pin_24)
- net SPIO_DIN: no longer J1.21 (Pin_21)
- net SPIO_DOUT: no longer J1.19 (Pin_19)
- net SPIO_SCL: no longer J1.23 (Pin_23)
- net UART0_RX: no longer J1.10 (Pin_10)
- net UART0_TX: no longer J1.8 (Pin_8)
- net UART1_RX: no longer J1.11 (Pin_11)
- net UART1_TX: no longer J1.7 (Pin_7)
- net at U4.18 (VBUS_VS_DISCH): now also R5.1
- new net GPIO_A_O: J1.13 (Pin_13)
- new net GPIO_B_O: J1.15 (Pin_15)
- new net GPIO_C_O: J1.16 (Pin_16)
- new net GPIO_D_O: J1.18 (Pin_18)
- new net GPIO_E_O: J1.22 (Pin_22)
- new net GPIO_F_O: J1.37 (Pin_37)
- new net GPIO_G_O: J1.29 (Pin_29)
- new net GPIO_H_O: J1.31 (Pin_31)
- new net GPIO_I_O: J1.33 (Pin_33)
- new net GPIO_J_O: J1.35 (Pin_35)
- new net GPIO_K_O: J1.38 (Pin_38)
- new net GPIO_L_O: J1.40 (Pin_40)
- new net I2C0_SCL_O: J1.28 (Pin_28)
- new net I2C0_SDA_O: J1.27 (Pin_27)
- new net I2C1_SCL_O: J1.5 (Pin_5)
- new net I2C1_SDA_O: J1.3 (Pin_3)
- new net SPIO_CS_O: J1.24 (Pin_24)
- new net SPIO_DIN_O: J1.21 (Pin_21)
- new net SPIO_DOUT_O: J1.19 (Pin_19)
- new net SPIO_SCL_O: J1.23 (Pin_23)
- new net UART0_RX_O: J1.10 (Pin_10)
- new net UART0_TX_O: J1.8 (Pin_8)
- new net UART1_RX_O: J1.11 (Pin_11)
- new net UART1_TX_O: J1.7 (Pin_7)
Other:
- note added: "Buttons\n"
- note added: "USB C"
- moved on the sheet: SW1, SW2
