File: Ultra96-IO-Mezzanine/Ultra96-IO-Mezzanine.kicad_pcb (KiCad board)
At the start: 2 copper layers, 85 x 54 mm, 4 parts, among them P1 CONN_02X20, P2 CONN_02X20, P3 CONN_02X30

Commit message: Changes
Parts:
- added D3: SP0503BAHT, Package_TO_SOT_SMD:SOT-143, F.Cu at (133.0, 122.9)
- added J1: USB_C_Receptacle_USB2.0, Connector_USB:USB_C_Receptacle_HRO_TYPE-C-31-M-12, F.Cu at (158.4, 102.5)
- added U2: CP2102N-A01-GQFN24, Package_DFN_QFN:QFN-24-1EP_4x4mm_P0.5mm_EP2.6x2.6mm, F.Cu at (152.3, 110.8)
- added U3: TXS0108EPW, Package_SO:TSSOP-20_4.4x6.5mm_P0.65mm, F.Cu at (115.9, 113.5)
Routing:
- net +1V8: track 0.00 -> 38.8 mm
- net GND: track 0.00 -> 14.4 mm
- net D-: track 0.00 -> 14.1 mm, vias 0 -> 2
- net D+: track 0.00 -> 13.5 mm
- net SYS_DCIN: track 0.00 -> 2.00 mm
- added copper zone on F.Cu, net GND
Other:
- net class Default: clearance 0 -> 0.1
- rule trace_clearance: 0 -> 0.1

Commit message: Progress
Parts:
- added U1: TXS0104ERGYR, BGA:Texas_DSBGA-10_1.36x1.86mm_Layout3x4_P0.5mm, F.Cu at (164.8, 110.2)

Commit message: Further work on PCB
Parts:
- added H1: MountingHole, 96boards:Hole_2.5MM, F.Cu at (104.0, 111.8)
- added H2: MountingHole, 96boards:Hole_2.5MM, F.Cu at (162.0, 111.8)
- added J2: Conn_01x08_Female, Connector_PinHeader_2.54mm:PinHeader_1x08_P2.54mm_Vertical, F.Cu at (181.0, 111.0)
- added J3: USB_C_Receptacle_USB2.0, Connector_USB:USB_C_Receptacle_HRO_TYPE-C-31-M-12, F.Cu at (169.7, 151.2)
- added P1: CONN_02X20, Connector_PinHeader_2.54mm:PinHeader_2x20_P2.54mm_Vertical, F.Cu at (133.0, 111.8)
- added U4: STUSB4500QTR, Package_DFN_QFN:QFN-24-1EP_4x4mm_P0.5mm_EP2.7x2.7mm, F.Cu at (156.0, 131.6)
- U1: footprint BGA:Texas_DSBGA-10_1.36x1.86mm_Layout3x4_P0.5mm -> Package_DFN_QFN:Texas_S-PVQFN-N14_ThermalVias
- U3: footprint Package_SO:TSSOP-20_4.4x6.5mm_P0.65mm -> LevelShifter:QFN50P450X350X100-21N
- moved J1 48.8 mm to (155.9, 151.3), turned to 0 degrees
- moved D3 33.9 mm to (159.9, 143.5), turned to 270 degrees
- moved U1 32.5 mm to (169.3, 78.0)
- moved U2 27.4 mm to (170.4, 131.4)
- moved U3 8.08 mm to (113.0, 121.0), turned to 90 degrees
- renumbered P3 to P2, P2 to P3
Connections:
- J1 pad A5: Net-(J1-PadA5) -> CC1
- J1 pad A6: D+ -> Net-(J1-PadA6)
- J1 pad A7: D- -> Net-(J1-PadA7)
- J1 pad B5: Net-(J1-PadB5) -> CC2
- J1 pad B6: D+ -> Net-(J1-PadB6)
- J1 pad B7: D- -> Net-(J1-PadB7)
- U3 pad 1: Net-(U3-Pad1) -> I2C0_SDA
- U3 pad 12: Net-(U3-Pad12) -> SPIO_SCL_RPI
- U3 pad 13: Net-(U3-Pad13) -> SPIO_DIN_RPI
- U3 pad 14: Net-(U3-Pad14) -> SPIO_DOUT_RPI
- U3 pad 15: Net-(U3-Pad15) -> GPIO_D_RPI
- U3 pad 16: Net-(U3-Pad16) -> GPIO_C_RPI
- U3 pad 17: Net-(U3-Pad17) -> GPIO_A_RPI
- U3 pad 18: Net-(U3-Pad18) -> I2C0_SCL_RPI
- U3 pad 20: Net-(U3-Pad20) -> I2C0_SDA_RPI
- U3 pad 3: Net-(U3-Pad3) -> I2C0_SCL
- U3 pad 4: Net-(U3-Pad4) -> GPIO_A
- U3 pad 5: Net-(U3-Pad5) -> GPIO_C
- U3 pad 6: Net-(U3-Pad6) -> GPIO_D
- U3 pad 7: Net-(U3-Pad7) -> SPIO_DOUT
- U3 pad 8: Net-(U3-Pad8) -> SPIO_DIN
- U3 pad 9: Net-(U3-Pad9) -> SPIO_SCL
Routing:
- net +1V8: track 38.8 -> 0.00 mm
- net GND: track 14.4 -> 38.1 mm
- net VBUS: track 0.00 -> 14.9 mm
- net CC2: track 0.00 -> 14.6 mm
- net CC1: track 0.00 -> 14.2 mm
- net D-: track 14.1 -> 0.00 mm, vias 2 -> 0
- net D+: track 13.5 -> 0.00 mm
