File: Ultra96-IO-Mezzanine/Ultra96-IO-Mezzanine.kicad_pcb (KiCad board)
At the start: 2 copper layers, 85 x 54 mm, 43 parts, among them J1 USB_C_Receptacle_USB2.0, J2 Conn_01x08_Female, J3 USB_C_Receptacle_USB2.0, P1 CONN_02X20, P2 CONN_02X30, P3 CONN_02X20, Q1 STL6P3LLH6, SW1 SW_SP3T, U1 TXS0104ERGYR, U2 CP2102N-A01-GQFN24, U3 TXS0108EPW, U4 STUSB4500QTR, U5 TXS0108EPW

Commit message: Started wiring
Parts:
- removed U1: TXS0104ERGYR, Package_DFN_QFN:Texas_S-PVQFN-N14_ThermalVias
- added PWR: SW_Push_Open, Button_Switch_SMD:SW_Push_1P1T_NO_Vertical_Wuerth_434133025816, F.Cu at (103.7, 121.4)
- added RST: SW_Push_Open, Button_Switch_SMD:SW_Push_1P1T_NO_Vertical_Wuerth_434133025816, F.Cu at (103.6, 127.6)
- added U6: TXS0108EPW, LevelShifter:QFN50P450X350X100-21N, F.Cu at (128.5, 119.9)
- added U7: TXS0108EPW, LevelShifter:QFN50P450X350X100-21N, F.Cu at (136.5, 119.9)
- 5v | 3v3 | 1v8: renamed from SW1
- moved 5v | 3v3 | 1v8 72.2 mm to (170.3, 101.9), turned to 180 degrees
- moved R2 44.3 mm to (164.3, 82.8)
- moved D2 42.4 mm to (162.1, 102.4), turned to 90 degrees
- moved C1 42.1 mm to (147.9, 79.9)
- moved C4 42.1 mm to (146.5, 77.0)
- moved C6 42.1 mm to (150.9, 74.0)
- moved R1 42.1 mm to (155.3, 77.0)
- moved R10 42.1 mm to (150.9, 77.0)
- moved R3 42.1 mm to (152.3, 79.9)
- moved R8 42.1 mm to (155.3, 74.0)
- moved R9 42.1 mm to (146.5, 74.0)
- moved D1 33.1 mm to (159.4, 102.4), turned to 90 degrees
- moved C8 32.5 mm to (156.9, 93.1)
- moved D4 32.5 mm to (155.5, 90.1)
- moved C3 31.2 mm to (104.0, 116.6), turned to 270 degrees
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Routing:
- net I2C0_SDA_RPI: track 0.00 -> 118.1 mm, vias 0 -> 7
- net +1V8: track 0.00 -> 87.1 mm, vias 0 -> 7
- net GND: track 148.2 -> 225.6 mm, vias 8 -> 23
- net I2C0_SCL_RPI: track 0.00 -> 70.1 mm, vias 0 -> 5
- net UART0_RTS: track 0.00 -> 64.6 mm, vias 0 -> 1
- net UART0_RX: track 0.00 -> 61.3 mm, vias 0 -> 1
- net UART0_TX: track 0.00 -> 61.1 mm, vias 0 -> 1
- net GPIO_D: track 0.00 -> 59.7 mm, vias 0 -> 9
- net UART0_CTS: track 0.00 -> 59.2 mm, vias 0 -> 2
- net GPIO_C: track 0.00 -> 54.7 mm, vias 0 -> 5
- net SPIO_DOUT: track 0.00 -> 51.7 mm, vias 0 -> 6
- net GPIO_A: track 0.00 -> 51.1 mm, vias 0 -> 4
- net VCCB: track 0.00 -> 49.1 mm, vias 0 -> 6
- net GPIO_L_RPI: track 0.00 -> 45.6 mm
- net GPIO_J_RPI: track 0.00 -> 44.5 mm
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Other:
- outline, holes or cut-outs redrawn

Commit message: 3 left
Parts:
- removed REF**: 96Boards CE Outline Standard, 96boards:96Boards_CE_outline_std
- 5v|3v3|1v8: renamed from 5v | 3v3 | 1v8
- U5, U6, U7: footprint LevelShifter:QFN50P450X350X100-21N -> Ultra96:QFN50P450X350X100-21N
- moved Q1 44.9 mm to (176.3, 108.1)
- moved R6 27.2 mm to (167.3, 120.5)
- moved C5 17.9 mm to (107.1, 139.6)
- moved R7 16.0 mm to (135.9, 145.5)
- moved D7 15.5 mm to (164.6, 133.3)
- moved C2 15.3 mm to (123.7, 146.1)
- moved C7 15.0 mm to (128.0, 146.3)
- moved D6 13.1 mm to (111.0, 143.7)
- moved U7 12.5 mm to (148.6, 123.1)
- moved D5 10.2 mm to (161.8, 133.3)
- moved C9 10.00 mm to (113.2, 138.7)
- moved U6 8.71 mm to (136.6, 123.1)
- moved U5 5.20 mm to (124.6, 123.1)
- moved U3 3.20 mm to (112.6, 123.1)
- renumbered J1 to PWR, J3 to UART
Routing:
- net PCM_DO_RPI: track 0.00 -> 92.6 mm, vias 0 -> 4
- net PCM_DI_RPI: track 0.00 -> 91.6 mm, vias 0 -> 4
- net PCM_FS_RPI: track 0.00 -> 90.2 mm, vias 0 -> 5
- net GPIO_L_RPI: track 45.6 -> 128.6 mm, vias 0 -> 5
- net GPIO_L: track 0.00 -> 82.2 mm, vias 0 -> 3
- net GPIO_J_RPI: track 44.5 -> 123.4 mm, vias 0 -> 7
- net +1V8: track 87.1 -> 158.3 mm, vias 7 -> 18
- net I2C1_SCL_RPI: track 0.00 -> 65.7 mm, vias 0 -> 8
- net GPIO_J: track 0.00 -> 61.0 mm, vias 0 -> 9
- net GND: track 225.6 -> 282.7 mm, vias 23 -> 36
- net GPIO_B: track 0.00 -> 53.1 mm, vias 0 -> 9
- net VCCB: track 49.1 -> 98.1 mm, vias 6 -> 19
- net UART1_TX: track 0.00 -> 46.4 mm, vias 0 -> 6
- net UART1_RX: track 0.00 -> 44.9 mm, vias 0 -> 9
- net PCM_DI: track 0.00 -> 38.7 mm, vias 0 -> 7
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- added copper zone on B.Cu, net GND

Commit message: All levelshifters routed
Parts:
- moved C9 39.3 mm to (152.5, 137.6), turned to 180 degrees
- moved R7 26.6 mm to (161.2, 137.3)
- moved Q1 24.2 mm to (163.0, 128.4)
- moved D4 12.6 mm to (152.3, 102.4), turned to 270 degrees
- moved C8 11.1 mm to (150.5, 102.1), turned to 270 degrees
Routing:
- net GPIO_K: track 2.96 -> 47.7 mm, vias 1 -> 5
- net GPIO_I: track 4.33 -> 35.8 mm, vias 1 -> 4
- net +3V3: track 33.2 -> 63.9 mm, vias 0 -> 2
- net GPIO_G: track 5.15 -> 31.5 mm, vias 1 -> 6
- net GND: track 282.7 -> 307.8 mm, vias 36 -> 31
- net +5V: track 33.8 -> 57.4 mm
- net I2C1_SCL_RPI: track 65.7 -> 69.4 mm
- net UART1_TX: track 46.4 -> 48.7 mm
- net VCCB: track 98.1 -> 100.5 mm
- net GPIO_B_RPI: track 15.7 -> 17.6 mm
- net GPIO_J: track 61.0 -> 62.8 mm
- net GPIO_H: track 37.9 -> 39.5 mm
- net PCM_DO: track 38.5 -> 36.9 mm
- net PCM_DI: track 38.7 -> 37.2 mm
- net I2C1_SCL: track 36.8 -> 35.4 mm
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
Commit message: Finished routing
Parts:
- moved C4 63.5 mm to (178.5, 131.8)
- moved R3 59.5 mm to (177.1, 134.1), turned to 180 degrees
- moved R1 57.9 mm to (174.6, 131.5), turned to 180 degrees
- moved C5 56.8 mm to (163.8, 139.8), turned to 180 degrees
- moved C6 55.5 mm to (148.4, 129.5), turned to 180 degrees
- moved R8 52.2 mm to (164.3, 125.5), turned to 180 degrees
- moved C1 51.2 mm to (174.5, 123.7), turned to 180 degrees
- moved R2 46.2 mm to (173.7, 128.0), turned to 0 degrees
- moved R9 43.5 mm to (165.4, 113.3), turned to 180 degrees
- moved D6 41.5 mm to (152.6, 144.4), turned to 180 degrees
- moved C2 36.6 mm to (159.8, 139.8)
- moved C7 34.2 mm to (155.3, 125.7), turned to 90 degrees
- moved R10 29.9 mm to (152.3, 106.8), turned to 270 degrees
- moved R7 18.6 mm to (166.7, 119.5)
- moved Q1 12.5 mm to (166.6, 116.5)
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Routing:
- net +3V3: track 63.9 -> 207.0 mm, vias 2 -> 12
- net +1V8: track 158.6 -> 265.1 mm, vias 20 -> 27
- net +5V: track 57.4 -> 163.6 mm, vias 0 -> 9
- net VBUS: track 0.00 -> 61.7 mm, vias 0 -> 2
- net VBUS_PWR: track 21.1 -> 63.8 mm, vias 0 -> 7
- net SYS_DCIN: track 2.00 -> 40.7 mm, vias 2 -> 6
- net GND: track 307.8 -> 346.4 mm, vias 31 -> 50
- net Net-(Q1-Pad4): track 0.00 -> 38.3 mm, vias 0 -> 4
- net Net-(R9-Pad2): track 0.00 -> 24.9 mm, vias 0 -> 4
- net I2C0_SDA_RPI: track 87.1 -> 111.7 mm, vias 3 -> 7
- net Net-(R6-Pad1): track 0.00 -> 15.9 mm, vias 0 -> 5
- net Net-(R8-Pad2): track 0.00 -> 10.9 mm, vias 0 -> 2
- net CC1: track 14.4 -> 24.4 mm
- net I2C0_SCL_RPI: track 107.9 -> 116.6 mm, vias 4 -> 7
- net Net-(C7-Pad1): track 0.00 -> 6.68 mm
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
Commit message: Tidying
Parts:
- added REF**: 96Boards CE Outline Standard, 96boards:96Boards_CE_outline_std, F.Cu at (100.0, 154.0)
- moved R3 2.76 mm to (175.6, 136.4)
Routing:
- net PCM_DO_RPI: track 92.4 -> 89.1 mm
- net PCM_DI_RPI: track 91.6 -> 88.9 mm
- net PCM_FS_RPI: track 90.6 -> 88.2 mm
- net GPIO_L_RPI: track 128.9 -> 126.6 mm
- net PCM_FS: track 44.3 -> 42.1 mm
- net GPIO_J_RPI: track 123.3 -> 121.5 mm
- net I2C1_SCL_RPI: track 69.4 -> 68.5 mm
- net GND: track 346.4 -> 345.5 mm, vias 50 -> 51
- net I2C1_SDA_RPI: track 56.5 -> 56.0 mm
Other:
- board text removed: "This is a template for a 96Boards CE Standard size mezzanine PCB. It uses the 96Boards_CE_outline_std footprint to place the mounting holes, show the connector locations, and board outline. The outline footprint will help you ensure your components and connectors are placed correctly. If you want to use the extended board size then replace the outline footprint with the 96Boards_CE_outline_extd v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"

Commit message: Further tidying
Routing:
- net VBUS: track 61.7 -> 48.2 mm
- net +1V8: track 265.1 -> 255.1 mm
- net GND: track 345.5 -> 343.3 mm, vias 51 -> 50
