File: Ultra96-IO-Mezzanine/Ultra96-IO-Mezzanine.sch (KiCad schematic (older format))
At the start: 21 parts, among them P2 CONN_02X20, P3 CONN_02X30

Commit message: Changes
Parts:
- C1, C2, C3, C4: renamed from C?; symbol Device:C_Small -> Ultra96-IO-Mezzanine-rescue:C_Small-Device
- D1, D2: renamed from D?; symbol Device:LED -> Ultra96-IO-Mezzanine-rescue:LED-Device
- D3: renamed from D?; symbol Power_Protection:SP0503BAHT -> Ultra96-IO-Mezzanine-rescue:SP0503BAHT-Power_Protection
- J1: renamed from J?; footprint (none) -> Connector_USB:USB_C_Receptacle_HRO_TYPE-C-31-M-12; symbol Connector:USB_C_Receptacle_USB2.0 -> Ultra96-IO-Mezzanine-rescue:USB_C_Receptacle_USB2.0-Connector
- J2: renamed from J?; symbol Connector:Conn_01x08_Female -> Ultra96-IO-Mezzanine-rescue:Conn_01x08_Female-Connector
- R1, R2, R3, R4, R5: renamed from R?; symbol Device:R -> Ultra96-IO-Mezzanine-rescue:R-Device
- SW1: renamed from SW?; symbol Switch:SW_SP3T -> Ultra96-IO-Mezzanine-rescue:SW_SP3T-Switch
- U1: renamed from U?; symbol LevelShifer:TXS0104ERGYR -> Ultra96-IO-Mezzanine-rescue:TXS0104ERGYR-LevelShifer
- U2: renamed from U?; symbol Interface_USB:CP2102N-A01-GQFN24 -> Ultra96-IO-Mezzanine-rescue:CP2102N-A01-GQFN24-Interface_USB
- U3: renamed from U?; symbol Logic_LevelTranslator:TXS0108EPW -> Ultra96-IO-Mezzanine-rescue:TXS0108EPW-Logic_LevelTranslator
- gave numbers to parts that had none: 1

Commit message: Progress
Parts:
- U1: footprint QFN50P350X350X100-15N -> BGA:Texas_DSBGA-10_1.36x1.86mm_Layout3x4_P0.5mm
Connections:
- net CC1: now reaches J1.A5 (CC1)
- net CC2: now reaches J1.B5 (CC2)
- no-connect marks 15 -> 13
Other:
- moved on the sheet: C1, C2, J2, SW1
Changed lines of the file:
@@
 $Descr A4 11693 8268
 encoding utf-8
-Sheet 1 1
+Sheet 1 2
 Title "96Boards Mezzanine Project Template"
 Date "14 Aug 2015"
@@
 F 0 "U1" H 4350 2567 50  0000 C CNN
 F 1 "TXS0104ERGYR" H 4350 2476 50  0000 C CNN
-F 2 "QFN50P350X350X100-15N" H 4350 1700 50  0001 L BNN
+F 2 "BGA:Texas_DSBGA-10_1.36x1.86mm_Layout3x4_P0.5mm" H 4350 1700 50  0001 L BNN
 F 3 "TEXAS INSTRUMENTS" H 4350 1700 50  0001 L BNN
 F 4 "IPC 7351B" H 4350 1700 50  0001 L BNN "Field4"
@@
 RPi Header
 $Comp
-L Ultra96-IO-Mezzanine-rescue:USB_C_Receptacle_USB2.0-Connector J1
-U 1 1 5F45AEF7
-P 4050 6350
-F 0 "J1" H 4157 7217 50  0000 C CNN
-F 1 "USB_C_Receptacle_USB2.0" H 4157 7126 50  0000 C CNN
-F 2 "Connector_USB:USB_C_Receptacle_HRO_TYPE-C-31-M-12" H 4200 6350 50  0001 C CNN
-F 3 "https://www.usb.org/sites/default/files/documents/usb_type-c.zip" H 4200 6350 50  0001 C CNN
-	1    4050 6350
-	1    0    0    -1
-$EndComp
-$Comp
 L Ultra96-IO-Mezzanine-rescue:CP2102N-A01-GQFN24-Interface_USB U2
 U 1 1 5F45E042
@@
 L Ultra96-IO-Mezzanine-rescue:Conn_01x08_Female-Connector J2
 U 1 1 5F45EE80
-P 10050 4850
-F 0 "J2" H 10078 4826 50  0000 L CNN
-F 1 "Conn_01x08_Female" H 10078 4735 50  0000 L CNN
-F 2 "" H 10050 4850 50  0001 C CNN
-F 3 "~" H 10050 4850 50  0001 C CNN
-	1    10050 4850
+P 10950 4750
+F 0 "J2" H 10978 4726 50  0000 L CNN
+F 1 "Conn_01x08_Female" H 10978 4635 50  0000 L CNN
+F 2 "" H 10950 4750 50  0001 C CNN
+F 3 "~" H 10950 4750 50  0001 C CNN
+	1    10950 4750
 	1    0    0    -1
 $EndComp
@@
 Text GLabel 10600 5650 2    60   BiDi ~ 0
 D-
-Text GLabel 5350 5750 2    60   BiDi ~ 0
+Text GLabel 5850 5750 2    60   BiDi ~ 0
 VBUS
 Text GLabel 10600 5550 2    60   BiDi ~ 0
@@
 Wire Wire Line
 	5850 3150 5950 3150
-Wire Wire Line
-	4650 5750 4950 5750
 $Comp
 L Ultra96-IO-Mezzanine-rescue:C_Small-Device C1
 U 1 1 5F7EF19A
-P 4950 5850
-F 0 "C1" H 4800 5750 50  0000 L CNN
-F 1 "4.7uF" H 4650 5850 50  0000 L CNN
-F 2 "" H 4950 5850 50  0001 C CNN
-F 3 "~" H 4950 5850 50  0001 C CNN
-	1    4950 5850
-	1    0    0    -1
-$EndComp
-Connection ~ 4950 5750
-Wire Wire Line
-	4950 5750 5150 5750
+P 5450 5850
+F 0 "C1" H 5300 5750 50  0000 L CNN
+F 1 "4.7uF" H 5150 5850 50  0000 L CNN
+F 2 "" H 5450 5850 50  0001 C CNN
+F 3 "~" H 5450 5850 50  0001 C CNN
+	1    5450 5850
+	1    0    0    -1
+$EndComp
+Connection ~ 5450 5750
+Wire Wire Line
+	5450 5750 5650 5750
 $Comp
 L Ultra96-IO-Mezzanine-rescue:C_Small-Device C2
 U 1 1 5F7EF629
-P 5150 5850
-F 0 "C2" H 5200 5750 50  0000 L CNN
-F 1 "0.1uF" H 5250 5850 50  0000 L CNN
-F 2 "" H 5150 5850 50  0001 C CNN
-F 3 "~" H 5150 5850 50  0001 C CNN
-	1    5150 5850
-	1    0    0    -1
-$EndComp
-Connection ~ 5150 5750
-Wire Wire Line
-	5150 5750 5350 5750
-Wire Wire Line
-	5150 5950 5050 5950
+P 5650 5850
+F 0 "C2" H 5700 5750 50  0000 L CNN
+F 1 "0.1uF" H 5750 5850 50  0000 L CNN
+F 2 "" H 5650 5850 50  0001 C CNN
+F 3 "~" H 5650 5850 50  0001 C CNN
+	1    5650 5850
+	1    0    0    -1
+$EndComp
+Connection ~ 5650 5750
+Wire Wire Line
+	5650 5750 5850 5750
+Wire Wire Line
+	5650 5950 5550 5950
 $Comp
 L Ultra96-IO-Mezzanine-rescue:GND-power #PWR0119
 U 1 1 5F805C49
-P 5050 5950
-F 0 "#PWR0119" H 5050 5700 50  0001 C CNN
-F 1 "GND" H 5200 5900 50  0000 C CNN
-F 2 "" H 5050 5950 50  0001 C CNN
-F 3 "" H 5050 5950 50  0001 C CNN
-	1    5050 5950
-	1    0    0    -1
-$EndComp
-Connection ~ 5050 5950
-Wire Wire Line
-	5050 5950 4950 5950
-NoConn ~ 4650 5950
-NoConn ~ 4650 6050
+P 5550 5950
+F 0 "#PWR0119" H 5550 5700 50  0001 C CNN
+F 1 "GND" H 5700 5900 50  0000 C CNN
+F 2 "" H 5550 5950 50  0001 C CNN
+F 3 "" H 5550 5950 50  0001 C CNN
+	1    5550 5950
+	1    0    0    -1
+$EndComp
+Connection ~ 5550 5950
+Wire Wire Line
+	5550 5950 5450 5950
 NoConn ~ 4650 6850
 NoConn ~ 4650 6950
@@
 	7000 2200 7000 2250
 $Comp
+L Ultra96-IO-Mezzanine-rescue:+1V8-power #PWR0122
+U 1 1 5F912A15
+P 9800 6050
+F 0 "#PWR0122" H 9800 5900 50  0001 C CNN
+F 1 "+1V8" V 9800 6190 50  0000 C CNN
+F 2 "" H 9800 6050 60  0000 C CNN
+F 3 "" H 9800 6050 60  0000 C CNN
+	1    9800 6050
+	1    0    0    -1
+$EndComp
+$Comp
+L Ultra96-IO-Mezzanine-rescue:+3V3-power #PWR0123
+U 1 1 5F913548
+P 9950 6050
+F 0 "#PWR0123" H 9950 5900 50  0001 C CNN
+F 1 "+3V3" V 9965 6223 50  0000 C CNN
+F 2 "" H 9950 6050 50  0001 C CNN
+F 3 "" H 9950 6050 50  0001 C CNN
+	1    9950 6050
+	1    0    0    -1
+$EndComp
+$Comp
+L Ultra96-IO-Mezzanine-rescue:+5V-power #PWR0124
+U 1 1 5F913C41
+P 10100 6050
+F 0 "#PWR0124" H 10100 5900 50  0001 C CNN
+F 1 "+5V" V 10100 6190 50  0000 C CNN
+F 2 "" H 10100 6050 60  0000 C CNN
+F 3 "" H 10100 6050 60  0000 C CNN
+	1    10100 6050
+	1    0    0    -1
+$EndComp
+Wire Wire Line
+	9800 6050 9800 6150
+Wire Wire Line
+	9800 6150 9600 6150
+Wire Wire Line
+	9600 6250 9950 6250
+Wire Wire Line
+	9950 6250 9950 6050
+Wire Wire Line
+	9600 6350 10100 6350
+Wire Wire Line
+	10100 6350 10100 6050
+$Comp
+L Ultra96-IO-Mezzanine-rescue:USB_C_Receptacle_USB2.0-Connector J1
+U 1 1 5F45AEF7
+P 4050 6350
+F 0 "J1" H 4157 7217 50  0000 C CNN
+F 1 "USB_C_Receptacle_USB2.0" H 4157 7126 50  0000 C CNN
+F 2 "Connector_USB:USB_C_Receptacle_HRO_TYPE-C-31-M-12" H 4200 6350 50  0001 C CNN
+F 3 "https://www.usb.org/sites/default/files/documents/usb_type-c.zip" H 4200 6350 50  0001 C CNN
+	1    4050 6350
+	1    0    0    -1
+$EndComp
+Wire Wire Line
+	4650 5750 5450 5750
+Text GLabel 4900 5950 2    60   Output ~ 0
+CC1
+Wire Wire Line
+	4900 5950 4650 5950
+Text GLabel 4900 6050 2    60   Output ~ 0
+CC2
+Wire Wire Line
+	4900 6050 4650 6050
+Wire Wire Line
+	9100 6250 9200 6250
+Text GLabel 9100 6250 0    60   BiDi ~ 0
+VCCB
+$Comp
 L Ultra96-IO-Mezzanine-rescue:SW_SP3T-Switch SW1
 U 1 1 5F8FB7EE
-P 8450 5550
-F 0 "SW1" H 8450 5833 50  0000 C CNN
-F 1 "SW_SP3T" H 8450 5742 50  0000 C CNN
-F 2 "" H 7825 5725 50  0001 C CNN
-F 3 "~" H 7825 5725 50  0001 C CNN
-	1    8450 5550
-	1    0    0    -1
-$EndComp
-Text GLabel 8150 5550 0    60   BiDi ~ 0
-VCCB
-Wire Wire Line
-	8150 5550 8250 5550
-$Comp
-L Ultra96-IO-Mezzanine-rescue:+1V8-power #PWR0122
-U 1 1 5F912A15
-P 8850 5350
-F 0 "#PWR0122" H 8850 5200 50  0001 C CNN
-F 1 "+1V8" V 8850 5490 50  0000 C CNN
-F 2 "" H 8850 5350 60  0000 C CNN
-F 3 "" H 8850 5350 60  0000 C CNN
-	1    8850 5350
-	1    0    0    -1
-$EndComp
-$Comp
-L Ultra96-IO-Mezzanine-rescue:+3V3-power #PWR0123
-U 1 1 5F913548
-P 9000 5350
-F 0 "#PWR0123" H 9000 5200 50  0001 C CNN
-F 1 "+3V3" V 9015 5523 50  0000 C CNN
-F 2 "" H 9000 5350 50  0001 C CNN
-F 3 "" H 9000 5350 50  0001 C CNN
-	1    9000 5350
-	1    0    0    -1
-$EndComp
-$Comp
-L Ultra96-IO-Mezzanine-rescue:+5V-power #PWR0124
-U 1 1 5F913C41
-P 9150 5350
-F 0 "#PWR0124" H 9150 5200 50  0001 C CNN
-F 1 "+5V" V 9150 5490 50  0000 C CNN
-F 2 "" H 9150 5350 60  0000 C CNN
-F 3 "" H 9150 5350 60  0000 C CNN
-	1    9150 5350
-	1    0    0    -1
-$EndComp
-Wire Wire Line
-	8850 5350 8850 5450
-Wire Wire Line
-	8850 5450 8650 5450
-Wire Wire Line
-	8650 5550 9000 5550
-Wire Wire Line
-	9000 5550 9000 5350
-Wire Wire Line
-	8650 5650 9150 5650
-Wire Wire Line
-	9150 5650 9150 5350
+P 9400 6250
+F 0 "SW1" H 9400 6533 50  0000 C CNN
+F 1 "SW_SP3T" H 9400 6442 50  0000 C CNN
+F 2 "" H 8775 6425 50  0001 C CNN
+F 3 "~" H 8775 6425 50  0001 C CNN
+	1    9400 6250
+	1    0    0    -1
+$EndComp
+Text GLabel 1400 6800 0    60   BiDi ~ 0
+VBUS
+Wire Wire Line
+	1400 6800 1550 6800
+Text GLabel 1400 7000 0    60   Output ~ 0
+CC1
+Text GLabel 1400 7100 0    60   Output ~ 0
+CC2
+Wire Wire Line
+	1400 7000 1550 7000
+Wire Wire Line
+	1400 7100 1550 7100
+$Sheet
+S 1550 6700 650  850
+U 5F27C63F
+F0 "Power" 60
+F1 "power.sch" 60
+F2 "CC1" I L 1550 7000 60
+F3 "CC2" I L 1550 7100 60
+F4 "VBUS" I L 1550 6800 60
+$EndSheet
 $EndSCHEMATC

Commit message: Further work on PCB
Parts:
- added C5, C6, C7: 1uF, symbol Device:C_Small
- added H1, H2: MountingHole, 96boards:Hole_2.5MM, symbol Mechanical:MountingHole
- added J3: USB_C_Receptacle_USB2.0, Connector_USB:USB_C_Receptacle_HRO_TYPE-C-31-M-12, symbol Ultra96-IO-Mezzanine-rescue:USB_C_Receptacle_USB2.0-Connector
- added R6: 1K, symbol Device:R
- added TP1, TP2: TestPoint, symbol Connector:TestPoint
- added U4: STUSB4500QTR, Package_DFN_QFN:QFN-24-1EP_4x4mm_P0.5mm_EP2.7x2.7mm, symbol Interface_USB:STUSB4500QTR
- J2: footprint (none) -> Connector_PinHeader_2.54mm:PinHeader_1x08_P2.54mm_Vertical
- P1: footprint (none) -> Connector_PinHeader_2.54mm:PinHeader_2x20_P2.54mm_Vertical
- U1: footprint BGA:Texas_DSBGA-10_1.36x1.86mm_Layout3x4_P0.5mm -> Package_DFN_QFN:Texas_S-PVQFN-N14_ThermalVias
- U3: footprint Package_SO:TSSOP-20_4.4x6.5mm_P0.65mm -> LevelShifter:QFN50P450X350X100-21N
- renumbered P3 to P2, P2 to P3
Connections:
- net CC1: now also U4.1 (CC1DB), U4.2 (CC1)
- net CC2: now also U4.4 (CC2), U4.5 (CC2DB)
- net D+: now also J3.A6 (D+), J3.B6 (D+); no longer J1.A6 (D+), J1.B6 (D+)
- net D-: now also J3.A7 (D-), J3.B7 (D-); no longer J1.A7 (D-), J1.B7 (D-)
- net GND: now also J2.4 (Pin_4), C5.2, C6.2, C7.2, J3.A1 (GND), J3.A12 (GND), J3.B1 (GND), J3.B12 (GND), J3.S1 (SHIELD), U4.10 (GND), U4.12 (ADDR0), U4.13 (ADDR1), U4.25 (GND)
- net GPIO_A: now also U3.4 (A3)
- net GPIO_A_RPI: now also U3.17 (B3)
- net GPIO_C: now also U3.5 (A4)
- net GPIO_C_RPI: now also U3.16 (B4)
- net GPIO_D: now also U3.6 (A5)
- net GPIO_D_RPI: now also U3.15 (B5)
- net GPIO_I_RPI: now also J2.5 (Pin_5)
- net GPIO_J_RPI: now also J2.6 (Pin_6)
- net GPIO_K_RPI: now also J2.8 (Pin_8)
- net GPIO_L_RPI: now also J2.7 (Pin_7)
- net I2C0_SCL: now also U3.3 (A2)
- net I2C0_SCL_RPI: now also J2.1 (Pin_1), U3.18 (B2), TP1.1, U4.7 (SCL)
- net I2C0_SDA: now also U3.1 (A1)
- net I2C0_SDA_RPI: now also J2.2 (Pin_2), U3.20 (B1), TP2.1, U4.8 (SDA)
- net SPIO_DIN: now also U3.8 (A7)
- net SPIO_DIN_RPI: now also U3.13 (B7)
- net SPIO_DOUT: now also U3.7 (A6)
- net SPIO_DOUT_RPI: now also U3.14 (B6)
- net SPIO_SCL: now also U3.9 (A8)
- net SPIO_SCL_RPI: now also U3.12 (B8)
- net VBUS: now also C5.1, R6.2, U4.24 (VDD); no longer R1.1
- net VCCB: now also J2.3 (Pin_3)
- new net: R6.1, U4.18 (VBUS_VS_DISCH)
- new net: C7.1, U4.21 (VREG_1V2)
- new net: J3.A4 (VBUS), J3.A9 (VBUS), J3.B4 (VBUS), J3.B9 (VBUS)
- new net +2V8: C6.1, U4.23 (VREG_2V7)
Other:
- moved on the sheet: C1, C2, J1, P1, P2, P3, U3
