File: Ultra96-IO-Mezzanine/Ultra96-IO-Mezzanine.sch (KiCad schematic (older format))
At the start: 45 parts, among them J1 USB_C_Receptacle_USB2.0, J2 Conn_01x08_Female, J3 USB_C_Receptacle_USB2.0, P1 CONN_02X20, P2 CONN_02X30, P3 CONN_02X20, Q1 STL6P3LLH6, SW1 SW_SP3T, U1 TXS0104ERGYR, U2 CP2102N-A01-GQFN24, U3 TXS0108EPW, U4 STUSB4500QTR, U5 TXS0108EPW

Commit message: Started wiring
Parts:
- removed U1: TXS0104ERGYR, Package_DFN_QFN:Texas_S-PVQFN-N14_ThermalVias, symbol Ultra96-IO-Mezzanine-rescue:TXS0104ERGYR-LevelShifer
- SW2, SW3: renamed from SW?; footprint (none) -> Button_Switch_SMD:SW_Push_1P1T_NO_Vertical_Wuerth_434133025816
- gave numbers to parts that had none: 2
Connections:
- net GND: now also SW2.1 (A), SW3.1 (A)
- net GPIO_B: now also U7.3 (A2)
- net GPIO_B_RPI: now also U7.18 (B2)
- net PWR_BTN_N: now also SW2.2 (B)
- net RST_BTN_N: now also SW3.2 (B)
- net SPIO_CS: now also U7.1 (A1)
- net SPIO_CS_RPI: now also U7.20 (B1)
- net UART0_CTS: now also U7.6 (A5)
- net UART0_CTS_O: now also U7.15 (B5)
- net UART0_RTS: now also U7.7 (A6)
- net UART0_RTS_O: now also U7.14 (B6)
- net UART0_RX: now also U7.5 (A4)
- net UART0_RX_O: now also U7.16 (B4)
- net UART0_TX: now also U7.4 (A3)
- net UART0_TX_O: now also U7.17 (B3)
- no-connect marks 26 -> 32
Other:
- note removed: "UART0 Level Shifter"
Changed lines of the file:
@@
 Wire Notes Line
 	13150 600  13150 4250
-$Comp
-L Ultra96-IO-Mezzanine-rescue:GND-power #PWR07
-U 1 1 5F13E6D4
-P 2900 2550
-F 0 "#PWR07" H 2900 2300 50  0001 C CNN
-F 1 "GND" H 2900 2400 50  0000 C CNN
-F 2 "" H 2900 2550 60  0000 C CNN
-F 3 "" H 2900 2550 60  0000 C CNN
-	1    2900 2550
-	1    0    0    -1
-$EndComp
-Wire Wire Line
-	2900 2450 2900 2550
-Text GLabel 1500 1850 0    60   Output ~ 0
+Text GLabel 8250 3750 0    60   Output ~ 0
 UART0_TX
 Wire Wire Line
-	1500 1850 1600 1850
-Text GLabel 1500 1950 0    60   Input ~ 0
+	8250 3750 8350 3750
+Text GLabel 8250 3850 0    60   Input ~ 0
 UART0_RX
 Wire Wire Line
-	1500 1950 1600 1950
-Text GLabel 1500 2050 0    60   Input ~ 0
+	8250 3850 8350 3850
+Text GLabel 8250 3950 0    60   Input ~ 0
 UART0_CTS
 Wire Wire Line
-	1500 2050 1600 2050
-Text GLabel 1500 2150 0    60   Output ~ 0
+	8250 3950 8350 3950
+Text GLabel 8250 4050 0    60   Output ~ 0
 UART0_RTS
 Wire Wire Line
-	1500 2150 1600 2150
-$Comp
-L Ultra96-IO-Mezzanine-rescue:+5V-power #PWR010
-U 1 1 5F1655F2
-P 3100 1250
-F 0 "#PWR010" H 3100 1100 50  0001 C CNN
-F 1 "+5V" H 3200 1300 50  0000 C CNN
-F 2 "" H 3100 1250 50  0001 C CNN
-F 3 "" H 3100 1250 50  0001 C CNN
-	1    3100 1250
-	1    0    0    -1
-$EndComp
-Text GLabel 2900 1850 2    60   Output ~ 0
+	8250 4050 8350 4050
+Text GLabel 9350 3750 2    60   Output ~ 0
 UART0_TX_O
-Wire Wire Line
-	2900 1850 2800 1850
-Text GLabel 2900 1950 2    60   Input ~ 0
+Text GLabel 9350 3850 2    60   Input ~ 0
 UART0_RX_O
-Wire Wire Line
-	2900 1950 2800 1950
-Text GLabel 2900 2050 2    60   Input ~ 0
+Text GLabel 9350 3950 2    60   Input ~ 0
 UART0_CTS_O
-Wire Wire Line
-	2900 2050 2800 2050
-Text GLabel 2900 2150 2    60   Output ~ 0
+Text GLabel 9350 4050 2    60   Output ~ 0
 UART0_RTS_O
-Wire Wire Line
-	2900 2150 2800 2150
-$Comp
-L Ultra96-IO-Mezzanine-rescue:TXS0104ERGYR-LevelShifer U1
-U 1 1 5F19EA6D
-P 2200 1950
-F 0 "U1" H 2200 2817 50  0000 C CNN
-F 1 "TXS0104ERGYR" H 2200 2726 50  0000 C CNN
-F 2 "Package_DFN_QFN:Texas_S-PVQFN-N14_ThermalVias" H 2200 1950 50  0001 L BNN
-F 3 "TEXAS INSTRUMENTS" H 2200 1950 50  0001 L BNN
-F 4 "IPC 7351B" H 2200 1950 50  0001 L BNN "Field4"
-F 5 "H" H 2200 1950 50  0001 L BNN "Field5"
-	1    2200 1950
-	1    0    0    -1
-$EndComp
-Wire Wire Line
-	2950 1250 2950 1350
-$Comp
-L Ultra96-IO-Mezzanine-rescue:+1V8-power #PWR09
-U 1 1 5F143AFB
-P 2950 1250
-F 0 "#PWR09" H 2950 1100 50  0001 C CNN
-F 1 "+1V8" H 2800 1300 50  0000 C CNN
-F 2 "" H 2950 1250 60  0000 C CNN
-F 3 "" H 2950 1250 60  0000 C CNN
-	1    2950 1250
-	1    0    0    -1
-$EndComp
-Wire Wire Line
-	2800 1350 2950 1350
-Wire Wire Line
-	2800 1450 3100 1450
-Wire Wire Line
-	3100 1250 3100 1450
-Wire Wire Line
-	2900 2450 2800 2450
-$Comp
-L Ultra96-IO-Mezzanine-rescue:+1V8-power #PWR03
-U 1 1 5F1F21A8
-P 1500 1250
-F 0 "#PWR03" H 1500 1100 50  0001 C CNN
-F 1 "+1V8" H 1500 1390 50  0000 C CNN
-F 2 "" H 1500 1250 60  0000 C CNN
-F 3 "" H 1500 1250 60  0000 C CNN
-	1    1500 1250
-	1    0    0    -1
-$EndComp
-Wire Wire Line
-	1500 1250 1500 1650
-Wire Wire Line
-	1500 1650 1600 1650
-Text Notes 1750 950  0    60   ~ 0
-UART0 Level Shifter
 $Comp
 L 96boards:CONN_02X20 P1
@@
 	4800 600  4800 4800
 $Comp
-L Ultra96-IO-Mezzanine-rescue:TXS0108EPW-Logic_LevelTranslator U?
+L Ultra96-IO-Mezzanine-rescue:TXS0108EPW-Logic_LevelTranslator U6
 U 1 1 6087561F
 P 6050 3800
-F 0 "U?" H 6450 3050 50  0000 C CNN
+F 0 "U6" H 6450 3050 50  0000 C CNN
 F 1 "TXS0108EPW" H 6450 2950 50  0000 C CNN
 F 2 "LevelShifter:QFN50P450X350X100-21N" H 6050 3050 50  0001 C CNN
@@
 	6150 2950 6150 3100
 $Comp
-L Ultra96-IO-Mezzanine-rescue:+1V8-power #PWR?
+L Ultra96-IO-Mezzanine-rescue:+1V8-power #PWR0121
 U 1 1 60968362
 P 5950 2950
-F 0 "#PWR?" H 5950 2800 50  0001 C CNN
+F 0 "#PWR0121" H 5950 2800 50  0001 C CNN
 F 1 "+1V8" H 5950 3090 50  0000 C CNN
 F 2 "" H 5950 2950 60  0000 C CNN
@@
 	5950 3050 5950 3100
 $Comp
-L Ultra96-IO-Mezzanine-rescue:GND-power #PWR?
+L Ultra96-IO-Mezzanine-rescue:GND-power #PWR0122
 U 1 1 609E325F
 P 6050 4650
-F 0 "#PWR?" H 6050 4400 50  0001 C CNN
+F 0 "#PWR0122" H 6050 4400 50  0001 C CNN
 F 1 "GND" H 6050 4500 50  0000 C CNN
 F 2 "" H 6050 4650 60  0000 C CNN
@@
 GPIO_F
 $Comp
-L Switch:SW_Push_Open SW?
+L Switch:SW_Push_Open SW2
 U 1 1 60B20626
 P 11350 4250
-F 0 "SW?" H 11350 4465 50  0000 C CNN
+F 0 "SW2" H 11350 4465 50  0000 C CNN
 F 1 "SW_Push_Open" H 11350 4374 50  0000 C CNN
-F 2 "" H 11350 4450 50  0001 C CNN
+F 2 "Button_Switch_SMD:SW_Push_1P1T_NO_Vertical_Wuerth_434133025816" H 11350 4450 50  0001 C CNN
 F 3 "~" H 11350 4450 50  0001 C CNN
 	1    11350 4250
@@
 $EndComp
 $Comp
-L Switch:SW_Push_Open SW?
+L Switch:SW_Push_Open SW3
 U 1 1 60B20916
 P 11350 4700
-F 0 "SW?" H 11350 4915 50  0000 C CNN
+F 0 "SW3" H 11350 4915 50  0000 C CNN
 F 1 "SW_Push_Open" H 11350 4824 50  0000 C CNN
-F 2 "" H 11350 4900 50  0001 C CNN
+F 2 "Button_Switch_SMD:SW_Push_1P1T_NO_Vertical_Wuerth_434133025816" H 11350 4900 50  0001 C CNN
 F 3 "~" H 11350 4900 50  0001 C CNN
 	1    11350 4700
@@
 $EndComp
 $Comp
-L Ultra96-IO-Mezzanine-rescue:TXS0108EPW-Logic_LevelTranslator U?
+L Ultra96-IO-Mezzanine-rescue:TXS0108EPW-Logic_LevelTranslator U7
 U 1 1 60B5F573
 P 8750 3850
-F 0 "U?" H 9150 3100 50  0000 C CNN
+F 0 "U7" H 9150 3100 50  0000 C CNN
 F 1 "TXS0108EPW" H 9150 3000 50  0000 C CNN
 F 2 "LevelShifter:QFN50P450X350X100-21N" H 8750 3100 50  0001 C CNN
@@
 $EndComp
 $Comp
-L Ultra96-IO-Mezzanine-rescue:GND-power #PWR?
+L Ultra96-IO-Mezzanine-rescue:GND-power #PWR0123
 U 1 1 60B604BC
 P 8750 4650
-F 0 "#PWR?" H 8750 4400 50  0001 C CNN
+F 0 "#PWR0123" H 8750 4400 50  0001 C CNN
 F 1 "GND" H 8750 4500 50  0000 C CNN
 F 2 "" H 8750 4650 60  0000 C CNN
@@
 	8850 2900 8850 3150
 $Comp
-L Ultra96-IO-Mezzanine-rescue:+1V8-power #PWR?
+L Ultra96-IO-Mezzanine-rescue:+1V8-power #PWR0124
 U 1 1 60BDA8DF
 P 8650 2900
-F 0 "#PWR?" H 8650 2750 50  0001 C CNN
+F 0 "#PWR0124" H 8650 2750 50  0001 C CNN
 F 1 "+1V8" H 8650 3040 50  0000 C CNN
 F 2 "" H 8650 2900 60  0000 C CNN
@@
 Wire Wire Line
 	5450 4200 5650 4200
+Text GLabel 9350 3550 2    60   Input ~ 0
+SPIO_CS_RPI
+Text GLabel 9350 3650 2    60   Input ~ 0
+GPIO_B_RPI
+Wire Wire Line
+	9150 3750 9350 3750
+Wire Wire Line
+	9150 3850 9350 3850
+Wire Wire Line
+	9150 3950 9350 3950
+Wire Wire Line
+	9150 4050 9350 4050
+Wire Wire Line
+	9350 3650 9150 3650
+Wire Wire Line
+	9350 3550 9150 3550
+Text GLabel 8250 3650 0    60   Input ~ 0
+GPIO_B
+Text GLabel 8250 3550 0    60   Input ~ 0
+SPIO_CS
+Wire Wire Line
+	8350 3550 8250 3550
+Wire Wire Line
+	8250 3650 8350 3650
+NoConn ~ 9150 4150
+NoConn ~ 9150 4250
+NoConn ~ 8350 4150
+NoConn ~ 8350 4250
+Text GLabel 11950 4250 2    60   Input ~ 0
+PWR_BTN_N
+Text GLabel 11950 4700 2    60   Input ~ 0
+RST_BTN_N
+Wire Wire Line
+	11950 4250 11550 4250
+Wire Wire Line
+	11950 4700 11550 4700
+$Comp
+L Ultra96-IO-Mezzanine-rescue:GND-power #PWR0125
+U 1 1 61598EB7
+P 10850 4350
+F 0 "#PWR0125" H 10850 4100 50  0001 C CNN
+F 1 "GND" H 10850 4200 50  0000 C CNN
+F 2 "" H 10850 4350 60  0000 C CNN
+F 3 "" H 10850 4350 60  0000 C CNN
+	1    10850 4350
+	1    0    0    -1
+$EndComp
+Wire Wire Line
+	11150 4250 10850 4250
+Wire Wire Line
+	10850 4250 10850 4350
+$Comp
+L Ultra96-IO-Mezzanine-rescue:GND-power #PWR0126
+U 1 1 615DE338
+P 10850 4800
+F 0 "#PWR0126" H 10850 4550 50  0001 C CNN
+F 1 "GND" H 10850 4650 50  0000 C CNN
+F 2 "" H 10850 4800 60  0000 C CNN
+F 3 "" H 10850 4800 60  0000 C CNN
+	1    10850 4800
+	1    0    0    -1
+$EndComp
+Wire Wire Line
+	11150 4700 10850 4700
+Wire Wire Line
+	10850 4700 10850 4800
+NoConn ~ 7700 6250
+NoConn ~ 7700 7450
 $EndSCHEMATC

Commit message: Tidy up schematic
Parts:
- added D10, D8, D9: LED, LED_SMD:LED_0805_2012Metric, symbol Ultra96-IO-Mezzanine-rescue:LED-Device
- added R11, R12, R13: 1K, Resistor_SMD:R_0805_2012Metric, symbol Device:R_Small
- Q1: symbol STL6P3LLH6:STL6P3LLH6 -> Ultra96-IO-Mezzanine-rescue:STL6P3LLH6-STL6P3LLH6
Connections:
- net +3V3: now also R11.1, R12.1, R13.1
- net at U4.14 (POWER_OK3): now also D10.1 (K)
- net at U4.15 (GPIO): now also D8.1 (K)
- net at U4.20 (POWER_OK2): now also D9.1 (K)
- new net: D8.2 (A), R11.2
- new net: D9.2 (A), R12.2
- new net: D10.2 (A), R13.2
- no-connect marks 32 -> 71
Changed lines of the file:
@@
 $EndComp
 $Comp
-L STL6P3LLH6:STL6P3LLH6 Q1
+L Ultra96-IO-Mezzanine-rescue:STL6P3LLH6-STL6P3LLH6 Q1
 U 1 1 5FCC6F93
 P 9750 5500
@@
 Wire Wire Line
 	2500 8450 2500 8650
-NoConn ~ 8900 6850
-NoConn ~ 8900 6950
 NoConn ~ 8900 7450
-NoConn ~ 8900 7550
 Wire Notes Line
 	10150 600  10150 4800
@@
 NoConn ~ 7700 6250
 NoConn ~ 7700 7450
+NoConn ~ 14550 950
+NoConn ~ 14550 1050
+NoConn ~ 14550 1150
+NoConn ~ 14550 1250
+NoConn ~ 14550 1350
+NoConn ~ 14550 1450
+NoConn ~ 14550 1650
+NoConn ~ 14550 1750
+NoConn ~ 14550 1950
+NoConn ~ 14550 2050
+NoConn ~ 14550 2250
+NoConn ~ 14550 2350
+NoConn ~ 14550 2550
+NoConn ~ 14550 2650
+NoConn ~ 14550 2850
+NoConn ~ 14550 2950
+NoConn ~ 14550 3150
+NoConn ~ 14550 3250
+NoConn ~ 14550 3450
+NoConn ~ 14550 3550
+NoConn ~ 14550 3750
+NoConn ~ 14550 3850
+NoConn ~ 15050 3650
+NoConn ~ 15050 3550
+NoConn ~ 15050 3350
+NoConn ~ 15050 3250
+NoConn ~ 15050 3050
+NoConn ~ 15050 2950
+NoConn ~ 15050 2750
+NoConn ~ 15050 2650
+NoConn ~ 15050 2550
+NoConn ~ 15050 2450
+NoConn ~ 15050 2250
+NoConn ~ 15050 2150
+NoConn ~ 15050 1950
+NoConn ~ 15050 1850
+NoConn ~ 15050 1650
+NoConn ~ 15050 1550
+NoConn ~ 15050 1350
+NoConn ~ 15050 1250
+NoConn ~ 15050 1050
+NoConn ~ 15050 950
+$Comp
+L Ultra96-IO-Mezzanine-rescue:LED-Device D8
+U 1 1 60235050
+P 9250 7550
+F 0 "D8" H 9243 7767 50  0000 C CNN
+F 1 "LED" H 9243 7676 50  0000 C CNN
+F 2 "LED_SMD:LED_0805_2012Metric" H 9250 7550 50  0001 C CNN
+F 3 "~" H 9250 7550 50  0001 C CNN
+	1    9250 7550
+	1    0    0    -1
+$EndComp
+$Comp
+L Device:R_Small R11
+U 1 1 60237D6E
+P 9650 7550
+F 0 "R11" V 9454 7550 50  0000 C CNN
+F 1 "1K" V 9545 7550 50  0000 C CNN
+F 2 "Resistor_SMD:R_0805_2012Metric" H 9650 7550 50  0001 C CNN
+F 3 "~" H 9650 7550 50  0001 C CNN
+	1    9650 7550
+	0    1    1    0
+$EndComp
+Wire Wire Line
+	8900 7550 9100 7550
+Wire Wire Line
+	9550 7550 9400 7550
+$Comp
+L Ultra96-IO-Mezzanine-rescue:+3V3-power #PWR0127
+U 1 1 60355339
+P 9950 7450
+F 0 "#PWR0127" H 9950 7300 50  0001 C CNN
+F 1 "+3V3" H 9965 7623 50  0000 C CNN
+F 2 "" H 9950 7450 50  0001 C CNN
+F 3 "" H 9950 7450 50  0001 C CNN
+	1    9950 7450
+	1    0    0    -1
+$EndComp
+Wire Wire Line
+	9950 7450 9950 7550
+Wire Wire Line
+	9950 7550 9750 7550
+$Comp
+L Ultra96-IO-Mezzanine-rescue:LED-Device D9
+U 1 1 6039CAD8
+P 9700 6350
+F 0 "D9" H 9693 6567 50  0000 C CNN
+F 1 "LED" H 9693 6476 50  0000 C CNN
+F 2 "LED_SMD:LED_0805_2012Metric" H 9700 6350 50  0001 C CNN
+F 3 "~" H 9700 6350 50  0001 C CNN
+	1    9700 6350
+	1    0    0    -1
+$EndComp
+$Comp
+L Ultra96-IO-Mezzanine-rescue:LED-Device D10
+U 1 1 6039D0EE
+P 9700 6600
+F 0 "D10" H 9693 6817 50  0000 C CNN
+F 1 "LED" H 9693 6726 50  0000 C CNN
+F 2 "LED_SMD:LED_0805_2012Metric" H 9700 6600 50  0001 C CNN
+F 3 "~" H 9700 6600 50  0001 C CNN
+	1    9700 6600
+	1    0    0    -1
+$EndComp
+$Comp
+L Device:R_Small R12
+U 1 1 6039D573
+P 10050 6350
+F 0 "R12" V 9854 6350 50  0000 C CNN
+F 1 "1K" V 9945 6350 50  0000 C CNN
+F 2 "Resistor_SMD:R_0805_2012Metric" H 10050 6350 50  0001 C CNN
+F 3 "~" H 10050 6350 50  0001 C CNN
+	1    10050 6350
+	0    1    1    0
+$EndComp
+$Comp
+L Device:R_Small R13
+U 1 1 6039D92C
+P 10050 6600
+F 0 "R13" V 9854 6600 50  0000 C CNN
+F 1 "1K" V 9945 6600 50  0000 C CNN
+F 2 "Resistor_SMD:R_0805_2012Metric" H 10050 6600 50  0001 C CNN
+F 3 "~" H 10050 6600 50  0001 C CNN
+	1    10050 6600
+	0    1    1    0
+$EndComp
+$Comp
+L Ultra96-IO-Mezzanine-rescue:+3V3-power #PWR0128
+U 1 1 6039DD64
+P 10350 6150
+F 0 "#PWR0128" H 10350 6000 50  0001 C CNN
+F 1 "+3V3" H 10365 6323 50  0000 C CNN
+F 2 "" H 10350 6150 50  0001 C CNN
+F 3 "" H 10350 6150 50  0001 C CNN
+	1    10350 6150
+	1    0    0    -1
+$EndComp
+Wire Wire Line
+	10350 6150 10350 6350
+Wire Wire Line
+	10350 6600 10150 6600
+Wire Wire Line
+	10150 6350 10350 6350
+Connection ~ 10350 6350
+Wire Wire Line
+	10350 6350 10350 6600
+Wire Wire Line
+	9950 6350 9850 6350
+Wire Wire Line
+	9950 6600 9850 6600
+Wire Wire Line
+	9550 6350 9300 6350
+Wire Wire Line
+	9300 6350 9300 6850
+Wire Wire Line
+	9300 6850 8900 6850
+Wire Wire Line
+	9550 6600 9400 6600
+Wire Wire Line
+	9400 6600 9400 6950
+Wire Wire Line
+	9400 6950 8900 6950
 $EndSCHEMATC
